File: pcb/fpga.kicad_sch (KiCad schematic)
At the start: 35 parts, among them J5 PINHD-1x7_ONIXJTAG-RevA, SW1 R-668049, U11 W25Q80EWUXIE, U12 DSC6011JI1A-050.0000, U8 LIF-MD6000-6UMG64I

Commit message: Rev. A initial design prior to fab comments
- BOM simplification
- Added my initials to the board
- Made the board more easy to panlize
Parts:
- added J3: SBH11-PBPC-D05-ST-BK, Connector_IDC:IDC-Header_2x05_P2.54mm_Vertical, symbol Connector_Generic:Conn_02x05_Odd_Even
- added JP1: Jumper_2_Open, jonnew:OE_SolderJumper-2_0201_Open_Pad, symbol Jumper:Jumper_2_Open
- C50: Voltage 10V -> (none)
- C51, C52: value 1.0uF -> 1uF
- D2: value LED -> SML-P11UTT86R
- TP9: now left out of the parts list
Connections:
- net +1V8: now also J3.4 (Pin_4)
- net DI_{Flash}/TMS: now also J3.5 (Pin_5)
- net DO_{Flash}/TCK: now also J3.1 (Pin_1)
- net GND: now also J3.10 (Pin_10), J3.2 (Pin_2)
- net SCLK_{Flash}/TDO: now also J3.3 (Pin_3)
- net TDI: now also J3.9 (Pin_9)
- net ~{CS}_{Flash}: now also J3.6 (Pin_6), JP1.2 (B); no longer U11.1 (~{CS})
- new net: JP1.1 (A), U11.1 (~{CS})
- no-connect marks 21 -> 23
Other:
- moved on the sheet: C58, D2, J5, R20, R21, R22, R25, U12

Commit message: Small changes before speedy fabrication
- This is revision A
Other:
- moved on the sheet: R21, R22
Changed lines of the file:
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@@
     (stroke (width 0) (type default) (color 0 0 0 0))
   )
-  (wire (pts (xy 250.19 179.07) (xy 250.19 180.34))
+  (wire (pts (xy 234.95 179.07) (xy 234.95 180.34))
     (stroke (width 0) (type default) (color 0 0 0 0))
   )
@@
     (stroke (width 0) (type default) (color 0 0 0 0))
   )
-  (wire (pts (xy 242.57 179.07) (xy 242.57 180.34))
+  (wire (pts (xy 227.33 179.07) (xy 227.33 180.34))
     (stroke (width 0) (type default) (color 0 0 0 0))
   )
@@
     (stroke (width 0) (type default) (color 0 0 0 0))
   )
-  (wire (pts (xy 242.57 194.31) (xy 180.34 194.31))
-    (stroke (width 0) (type default) (color 0 0 0 0))
-  )
-  (wire (pts (xy 242.57 187.96) (xy 242.57 194.31))
+  (wire (pts (xy 227.33 194.31) (xy 180.34 194.31))
+    (stroke (width 0) (type default) (color 0 0 0 0))
+  )
+  (wire (pts (xy 227.33 187.96) (xy 227.33 194.31))
     (stroke (width 0) (type default) (color 0 0 0 0))
   )
@@
     (stroke (width 0) (type default) (color 0 0 0 0))
   )
-  (wire (pts (xy 180.34 196.85) (xy 250.19 196.85))
-    (stroke (width 0) (type default) (color 0 0 0 0))
-  )
-  (wire (pts (xy 250.19 196.85) (xy 250.19 187.96))
+  (wire (pts (xy 180.34 196.85) (xy 234.95 196.85))
+    (stroke (width 0) (type default) (color 0 0 0 0))
+  )
+  (wire (pts (xy 234.95 196.85) (xy 234.95 187.96))
     (stroke (width 0) (type default) (color 0 0 0 0))
   )
@@
     (pin "1")
   )
-  (symbol (lib_id "power:+1V8") (at 250.19 179.07 0) (mirror y) (unit 1)
-    (in_bom yes) (on_board yes)
-    (property "Reference" "#PWR0106" (id 0) (at 250.19 182.88 0)
-      (effects (font (size 1.27 1.27)) hide)
-    )
-    (property "Value" "+1V8" (id 1) (at 250.19 175.26 0))
-    (property "Footprint" "" (id 2) (at 250.19 179.07 0)
-      (effects (font (size 1.27 1.27)) hide)
-    )
-    (property "Datasheet" "" (id 3) (at 250.19 179.07 0)
+  (symbol (lib_id "power:+1V8") (at 234.95 179.07 0) (mirror y) (unit 1)
+    (in_bom yes) (on_board yes)
+    (property "Reference" "#PWR0106" (id 0) (at 234.95 182.88 0)
+      (effects (font (size 1.27 1.27)) hide)
+    )
+    (property "Value" "+1V8" (id 1) (at 234.95 175.26 0))
+    (property "Footprint" "" (id 2) (at 234.95 179.07 0)
+      (effects (font (size 1.27 1.27)) hide)
+    )
+    (property "Datasheet" "" (id 3) (at 234.95 179.07 0)
       (effects (font (size 1.27 1.27)) hide)
     )
@@
     (pin "7")
   )
-  (symbol (lib_id "power:+1V8") (at 242.57 179.07 0) (mirror y) (unit 1)
-    (in_bom yes) (on_board yes)
-    (property "Reference" "#PWR0107" (id 0) (at 242.57 182.88 0)
-      (effects (font (size 1.27 1.27)) hide)
-    )
-    (property "Value" "+1V8" (id 1) (at 242.57 175.26 0))
-    (property "Footprint" "" (id 2) (at 242.57 179.07 0)
-      (effects (font (size 1.27 1.27)) hide)
-    )
-    (property "Datasheet" "" (id 3) (at 242.57 179.07 0)
+  (symbol (lib_id "power:+1V8") (at 227.33 179.07 0) (mirror y) (unit 1)
+    (in_bom yes) (on_board yes)
+    (property "Reference" "#PWR0107" (id 0) (at 227.33 182.88 0)
+      (effects (font (size 1.27 1.27)) hide)
+    )
+    (property "Value" "+1V8" (id 1) (at 227.33 175.26 0))
+    (property "Footprint" "" (id 2) (at 227.33 179.07 0)
+      (effects (font (size 1.27 1.27)) hide)
+    )
+    (property "Datasheet" "" (id 3) (at 227.33 179.07 0)
       (effects (font (size 1.27 1.27)) hide)
     )
@@
     (pin "G4")
   )
-  (symbol (lib_id "Device:R_US") (at 250.19 184.15 0) (unit 1)
-    (in_bom yes) (on_board yes)
-    (property "Reference" "R21" (id 0) (at 251.46 182.88 0)
-      (effects (font (size 1.27 1.27)) (justify left))
-    )
-    (property "Value" "4.7k" (id 1) (at 251.46 185.42 0)
-      (effects (font (size 1.27 1.27)) (justify left))
-    )
-    (property "Footprint" "Resistor_SMD:R_0201_0603Metric" (id 2) (at 251.206 184.404 90)
-      (effects (font (size 1.27 1.27)) hide)
-    )
-    (property "Datasheet" "~" (id 3) (at 250.19 184.15 0)
+  (symbol (lib_id "Device:R_US") (at 234.95 184.15 0) (unit 1)
+    (in_bom yes) (on_board yes)
+    (property "Reference" "R21" (id 0) (at 236.22 182.88 0)
+      (effects (font (size 1.27 1.27)) (justify left))
+    )
+    (property "Value" "4.7k" (id 1) (at 236.22 185.42 0)
+      (effects (font (size 1.27 1.27)) (justify left))
+    )
+    (property "Footprint" "Resistor_SMD:R_0201_0603Metric" (id 2) (at 235.966 184.404 90)
+      (effects (font (size 1.27 1.27)) hide)
+    )
+    (property "Datasheet" "~" (id 3) (at 234.95 184.15 0)
       (effects (font (size 1.27 1.27)) hide)
     )
@@
     (pin "1")
   )
-  (symbol (lib_id "Device:R_US") (at 242.57 184.15 0) (unit 1)
-    (in_bom yes) (on_board yes)
-    (property "Reference" "R22" (id 0) (at 243.84 182.88 0)
-      (effects (font (size 1.27 1.27)) (justify left))
-    )
-    (property "Value" "4.7k" (id 1) (at 243.84 185.42 0)
-      (effects (font (size 1.27 1.27)) (justify left))
-    )
-    (property "Footprint" "Resistor_SMD:R_0201_0603Metric" (id 2) (at 243.586 184.404 90)
-      (effects (font (size 1.27 1.27)) hide)
-    )
-    (property "Datasheet" "~" (id 3) (at 242.57 184.15 0)
-      (effects (font (size 1.27 1.27)) hide)
-    )
+  (symbol (lib_id "Device:R_US") (at 227.33 184.15 0) (unit 1)
+    (in_bom yes) (on_board yes)
+    (property "Reference" "R22" (id 0) (at 228.6 182.88 0)
+      (effects (font (size 1.27 1.27)) (justify left))
+    )
+    (property "Value" "4.7k" (id 1) (at 228.6 185.42 0)
+      (effects (font (size 1.27 1.27)) (justify left))
+    )
+    (property "Footprint" "Resistor_SMD:R_0201_0603Metric" (id 2) (at 228.346 184.404 90)
+      (effects (font (size 1.27 1.27)) hide)
+    )
+    (property "Datasheet" "~" (id 3) (at 227.33 184.15 0)
+      (effects (font (size 1.27 1.27)) hide)
+    )

Commit message: Start of revision B
- Address the following issues
1. The photodiode anode is on pin 3, not pin 2
2. No paste on coax connector
3. CRESET_B needs to come out to programming header
4. Need PU on CS line.
Parts:
- added R14: 4.7k, Resistor_SMD:R_0201_0603Metric, symbol Device:R_US
- C42, C43, C44, C45, C46, C47, C48, C49: TempCo (none) -> X7R; Voltage (none) -> 16V
- C50: TempCo (none) -> X5R; Voltage (none) -> 10V
- C51, C52, C53, C54, C55, C56, C57: TempCo (none) -> X5R; Voltage 10V -> 16V
- C58: TempCo (none) -> X7R; Voltage (none) -> 35V
- J5, JP1, TP9: DNP (none) -> DNP
Connections:
- net +1V8: now also R14.1
- net ~{CS}_{Flash}: now also R14.2
- net CRESET_{B}: now reaches R20.2, SW1.1, U8.E2 (CRESET_B)
- net CRESET_{B}: now also J3.8 (Pin_8)
- no-connect marks 23 -> 22
Other:
- title: Headstage-RHS2116 -> Headstage-64s
- moved on the sheet: SW1, TP9
